Commit message: Added thigh links

File: cheeto.urdf (robot description, URDF)
Before this commit: robot cheeto_quadruped, 13 links, 12 joints
Links:
- link base_link: geometry collision mesh filename=meshes/base.stl; visual mesh filename=meshes/base.stl
- link foot1: geometry collision sphere radius=0.02; visual mesh filename=meshes/foot.stl
- link foot2: geometry collision sphere radius=0.02; visual mesh filename=meshes/foot.stl
- link foot3: geometry collision sphere radius=0.02; visual mesh filename=meshes/foot.stl
- link foot4: geometry collision sphere radius=0.02; visual mesh filename=meshes/foot.stl
- link hip1: geometry collision mesh filename=meshes/hip.stl; visual mesh filename=meshes/hip.stl
- link hip2: geometry collision mesh filename=meshes/hip.stl; visual mesh filename=meshes/hip.stl
- link hip3: geometry collision mesh filename=meshes/hip.stl; visual mesh filename=meshes/hip.stl
- link hip4: geometry collision mesh filename=meshes/hip.stl; visual mesh filename=meshes/hip.stl
- link thigh1: geometry collision cylinder length=0.2 radius=0.015; visual mesh filename=meshes/thigh.stl
- link thigh2: geometry collision cylinder length=0.2 radius=0.015; visual mesh filename=meshes/thigh.stl
- link thigh3: geometry collision cylinder length=0.2 radius=0.015; visual mesh filename=meshes/thigh.stl
- link thigh4: geometry collision cylinder length=0.2 radius=0.015; visual mesh filename=meshes/thigh.stl
Joints:
- joint hip1_joint: origin xyz=0.15 0.1 0 rpy=0 0 0 -> xyz=86 46.5 24 rpy=0 0 0
- joint hip2_joint: origin xyz=0.15 -0.1 0 rpy=0 0 0 -> xyz=86 -46.5 24 rpy=0 0 0
- joint hip3_joint: origin xyz=-0.15 0.1 0 rpy=0 0 0 -> xyz=-86 46.5 24 rpy=0 0 3.14
- joint hip4_joint: origin xyz=-0.15 -0.1 0 rpy=0 0 0 -> xyz=-86 -46.5 24 rpy=0 0 3.14
- joint thigh1_joint: axis 1 0 0 -> 0 1 0; origin xyz=0 0 0 rpy=0 0 0 -> xyz=80 0 7 rpy=0 0 0
- joint thigh2_joint: axis 1 0 0 -> 0 1 0; origin xyz=0 0 0 rpy=0 0 0 -> xyz=80 0 7 rpy=0 0 0
- joint thigh3_joint: axis 1 0 0 -> 0 1 0; origin xyz=0 0 0 rpy=0 0 0 -> xyz=80 0 7 rpy=0 0 0
- joint thigh4_joint: axis 1 0 0 -> 0 1 0; origin xyz=0 0 0 rpy=0 0 0 -> xyz=80 0 7 rpy=0 0 0
